File: RoboBuddy_public/RoboBuddy.kicad_pcb (KiCad board)
At the start: 2 copper layers, 50 x 50 mm, 48 parts, among them J1 USB_B_Micro, J3 Micro_SD_Card, U1 RP2040, U2 NCP1117-3.3_SOT223, U3 W25Q128JVS, U4 LSM6DS3, Y1 ABM8-272-T3

Commit message: Add files via upload
Parts:
- removed ?: , 
- removed USB: TestPoint_Pad_D1.0mm, TestPoint:TestPoint_Pad_D1.0mm
- added 3.3v: TestPoint_THTPad_D1.0mm_Drill0.5mm, TestPoint:TestPoint_THTPad_D1.0mm_Drill0.5mm, F.Cu at (163.9, 72.5)
- added GND: TestPoint_THTPad_D1.0mm_Drill0.5mm, TestPoint:TestPoint_THTPad_D1.0mm_Drill0.5mm, F.Cu at (145.1, 72.5)
- added GND: TestPoint_THTPad_D1.0mm_Drill0.5mm, TestPoint:TestPoint_THTPad_D1.0mm_Drill0.5mm, F.Cu at (163.9, 74.9)
- added U4_SD0: TestPoint_THTPad_D1.0mm_Drill0.5mm, TestPoint:TestPoint_THTPad_D1.0mm_Drill0.5mm, F.Cu at (134.8, 103.9)
- added USB_Boot: TestPoint_THTPad_D1.0mm_Drill0.5mm, TestPoint:TestPoint_THTPad_D1.0mm_Drill0.5mm, F.Cu at (137.9, 74.0)
- C1, C2, C3, C4, C5, C6, C7, C8, C9: footprint Capacitor_SMD:C_0201_0603Metric -> Capacitor_SMD:C_0603_1608Metric
- C10: renamed from C11; footprint Capacitor_SMD:C_0201_0603Metric -> Capacitor_SMD:C_0603_1608Metric
- C11: renamed from C12; footprint Capacitor_SMD:C_0201_0603Metric -> Capacitor_SMD:C_0603_1608Metric
- C12: renamed from C13; footprint Capacitor_SMD:C_0201_0603Metric -> Capacitor_SMD:C_0603_1608Metric
- C13: renamed from C14; footprint Capacitor_SMD:C_0201_0603Metric -> Capacitor_SMD:C_0603_1608Metric
- C14: renamed from C15; footprint Capacitor_SMD:C_0201_0603Metric -> Capacitor_SMD:C_0603_1608Metric
- C15: renamed from C16; footprint Capacitor_SMD:C_0201_0603Metric -> Capacitor_SMD:C_0603_1608Metric
- R1, R10, R2, R3, R4, R5, R6, R7, R8, R9: footprint Resistor_SMD:R_0201_0603Metric -> Resistor_SMD:R_0603_1608Metric
- moved C2 20.9 mm to (155.9, 83.2), turned to 180 degrees
- moved U2 10.2 mm to (161.2, 82.7)
- moved Test 8.23 mm to (152.2, 109.1), turned to 180 degrees
- moved C1 7.90 mm to (155.9, 80.3), turned to 180 degrees
- moved R10 7.57 mm to (133.0, 91.0)
- moved R9 7.50 mm to (124.9, 91.1)
- moved C15 7.45 mm to (130.7, 91.1)
- moved R8 7.42 mm to (126.9, 91.1)
- moved R7 7.40 mm to (128.8, 91.1)
- moved R4 7.35 mm to (152.4, 81.5)
- moved GP9 7.12 mm to (127.2, 97.5)
- moved GP10 7.00 mm to (127.2, 99.9)
- moved GP11 7.00 mm to (127.2, 102.4)
- moved J1 6.57 mm to (154.4, 75.2)
- moved J2 6.40 mm to (129.4, 80.0)
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- renumbered J3 to J2
Routing:
- net /USB_D-: track 20.4 -> 6.24 mm
- net /USB_D+: track 19.1 -> 8.58 mm
- net /SDA_OLED: track 27.3 -> 17.7 mm
- net /RUN: track 28.4 -> 19.0 mm
- net /SCL_OLED: track 25.0 -> 16.0 mm
- net /SWD: track 29.5 -> 20.7 mm
- net /SWCLK: track 30.5 -> 21.9 mm
- net Net-(U1-USB_DM): track 2.20 -> 10.3 mm
- net /QSPI_SCLK: track 21.1 -> 13.1 mm
- net /MISO_SD: track 33.9 -> 25.9 mm
- net /QSPI_SD0: track 20.6 -> 12.8 mm
- net /speaker: track 15.0 -> 21.2 mm
- net GND: track 25.3 -> 19.2 mm, vias 27 -> 25
- net /SCL_GRYO/MOSI_SD: track 68.6 -> 62.5 mm
- net /QSPI_SD2: track 19.6 -> 14.5 mm
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Other:
- board size 50 x 50 mm -> 43.2 x 40.5 mm
- board text added: "RoboBud By: Ben"
- board text removed: "Powered by: RP2040"
- board text removed: "RoboBud By Ben"
